File: stm32io_mod.kicad_pcb (KiCad board)
At the start: 2 copper layers, 70.5 x 73.7 mm, 53 parts, among them J1 UART, M1 BluePill, Q1 BC858, Q2 BC858, Q3 BC858, Q4 BC858, SW1 button_1, SW2 button_2, SW3 button_3, SW4 button_4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

Commit message: Mejorando alguna rutas el PCB
Parts:
- removed the G*** at (126.7, 111.6)
- removed the REF** at (146.1, 92.2)
- removed the REF** at (169.5, 116.7)
- added REF**: OSHW-Logo2_7.3x6mm_Copper, Symbol:OSHW-Logo2_7.3x6mm_Copper, B.Cu at (167.4, 116.0)
- REF**: moved to B.Cu
- moved R9 15.1 mm to (137.2, 120.3), turned to 0 degrees
- moved R3 13.9 mm to (141.2, 118.8), turned to 0 degrees
- moved R8 10.1 mm to (137.2, 123.2), turned to 0 degrees
- moved R10 8.53 mm to (141.2, 121.8), turned to 0 degrees
- moved R7 4.51 mm to (141.2, 124.6), turned to 0 degrees
- moved D5 0.39 mm to (118.8, 104.8)
- moved D4 0.27 mm to (118.8, 109.4)
- moved D3 0.24 mm to (118.8, 114.0)
- moved D2 0.08 mm to (118.8, 118.6)
Connections:
- M1 pad 1: (no net) -> Net-(M1-Pad1)
- M1 pad 17: (no net) -> Net-(M1-Pad17)
- M1 pad 2: (no net) -> Net-(M1-Pad2)
- M1 pad 25: (no net) -> Net-(M1-Pad25)
- M1 pad 3: (no net) -> Net-(M1-Pad3)
- M1 pad 38: (no net) -> Net-(M1-Pad38)
- M1 pad 4: (no net) -> Net-(M1-Pad4)
Routing:
- net VCC: track 192.9 -> 269.8 mm, vias 0 -> 2
- net segC: track 1.78 -> 16.9 mm
- net segG: track 1.78 -> 16.5 mm
- net GND: track 42.4 -> 28.1 mm, vias 0 -> 2
- net Net-(R3-Pad1): track 22.2 -> 8.16 mm
- net Net-(R9-Pad1): track 21.1 -> 8.40 mm
- net segD: track 1.78 -> 9.80 mm
- net segP: track 1.78 -> 8.79 mm
- net Net-(R8-Pad1): track 18.4 -> 12.2 mm
- net Net-(R10-Pad1): track 19.6 -> 14.0 mm
- net Net-(R6-Pad1): track 23.0 -> 26.7 mm
- net Net-(D1-Pad3): track 53.3 -> 57.0 mm
- net Net-(D1-Pad1): track 54.6 -> 58.1 mm
- net Net-(D1-Pad4): track 53.2 -> 56.4 mm
- net Net-(D2-Pad1): track 49.2 -> 52.2 mm
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